File: Hardware/hikebuddy_dhauladhar/base.brd (EAGLE design)
At the start: 80 x 40 mm, 116 parts, among them J1 4P-SMD-2.0-90D, J2 4P-2.0-90D, J3 MF-CON-MICROUSB-RIGHT, J4 FH12-10S-0.5SH(1)(98), U11 MF-DSC-SOT233-BSS84, U3 MF-DSC-SOT233-MMBT3904, U4 MF-DSC-SOT233-MMBT3904, U9 MF-DSC-SOT233-BSS84

Commit message: last commit before starting V2
Parts:
- MOTOR+, MOTOR-, PIEZO+, PIEZO-: value (none) -> WIREPADSMD1,27-254
Changed lines of the file:
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@@
 <?xml version="1.0" encoding="utf-8"?>
 <!DOCTYPE eagle SYSTEM "eagle.dtd">
-<eagle version="9.3.1">
+<eagle version="9.5.1">
 <drawing>
 <settings>
-<setting alwaysvectorfont="yes"/>
+<setting alwaysvectorfont="no"/>
 <setting verticaltext="up"/>
 </settings>
@@
 <attribute name="PROD_ID" value="RES-00824" x="30" y="27.9" size="1.778" layer="27" font="vector" ratio="15" display="off"/>
 </element>
-<element name="PIEZO+" library="wirepad" library_urn="urn:adsk.eagle:library:412" package="SMD1,27-2,54" package3d_urn="urn:adsk.eagle:package:30839/1" value="" x="21.2" y="13.8" smashed="yes" rot="R180">
+<element name="PIEZO+" library="wirepad" library_urn="urn:adsk.eagle:library:412" package="SMD1,27-2,54" package3d_urn="urn:adsk.eagle:package:30839/1" value="WIREPADSMD1,27-254" x="21.2" y="13.8" smashed="yes" rot="R180">
 <attribute name="NAME" x="19.1" y="17.1" size="1.27" layer="25" rot="R270"/>
+<attribute name="POPULARITY" value="11" x="21.2" y="13.8" size="1.778" layer="27" rot="R180" display="off"/>
 <attribute name="VALUE" x="21.2" y="13.8" size="0.0254" layer="27" rot="R180"/>
 </element>
-<element name="PIEZO-" library="wirepad" library_urn="urn:adsk.eagle:library:412" package="SMD1,27-2,54" package3d_urn="urn:adsk.eagle:package:30839/1" value="" x="23.2" y="13.8" smashed="yes" rot="R180">
+<element name="PIEZO-" library="wirepad" library_urn="urn:adsk.eagle:library:412" package="SMD1,27-2,54" package3d_urn="urn:adsk.eagle:package:30839/1" value="WIREPADSMD1,27-254" x="23.2" y="13.8" smashed="yes" rot="R180">
 <attribute name="NAME" x="24" y="17.3" size="1.27" layer="25" rot="R270"/>
+<attribute name="POPULARITY" value="11" x="23.2" y="13.8" size="1.778" layer="27" rot="R180" display="off"/>
 <attribute name="VALUE" x="23.2" y="13.8" size="0.0254" layer="27" rot="R180"/>
 </element>
@@
 <attribute name="PROD_ID" value="RES-00824" x="30" y="31.7" size="1.778" layer="27" font="vector" ratio="15" display="off"/>
 </element>
-<element name="MOTOR+" library="wirepad" library_urn="urn:adsk.eagle:library:412" package="SMD1,27-2,54" package3d_urn="urn:adsk.eagle:package:30839/1" value="" x="21.2" y="22.9" smashed="yes" rot="R180">
+<element name="MOTOR+" library="wirepad" library_urn="urn:adsk.eagle:library:412" package="SMD1,27-2,54" package3d_urn="urn:adsk.eagle:package:30839/1" value="WIREPADSMD1,27-254" x="21.2" y="22.9" smashed="yes" rot="R180">
 <attribute name="NAME" x="19.2" y="26.5" size="1.27" layer="25" rot="R270"/>
+<attribute name="POPULARITY" value="11" x="21.2" y="22.9" size="1.778" layer="27" rot="R180" display="off"/>
 <attribute name="VALUE" x="21.2" y="22.9" size="0.0254" layer="27" rot="R180"/>
 </element>
-<element name="MOTOR-" library="wirepad" library_urn="urn:adsk.eagle:library:412" package="SMD1,27-2,54" package3d_urn="urn:adsk.eagle:package:30839/1" value="" x="23.2" y="22.9" smashed="yes" rot="R180">
+<element name="MOTOR-" library="wirepad" library_urn="urn:adsk.eagle:library:412" package="SMD1,27-2,54" package3d_urn="urn:adsk.eagle:package:30839/1" value="WIREPADSMD1,27-254" x="23.2" y="22.9" smashed="yes" rot="R180">
 <attribute name="NAME" x="24" y="26.3" size="1.27" layer="25" rot="R270"/>
+<attribute name="POPULARITY" value="11" x="23.2" y="22.9" size="1.778" layer="27" rot="R180" display="off"/>
 <attribute name="VALUE" x="23.2" y="22.9" size="0.0254" layer="27" rot="R180"/>
 </element>

Commit message: digikey_cs_v0
Parts:
- removed BATTERY: (no value), SparkFun-Connectors:JST-2-SMD
- removed C20: 0.22uF, SparkFun-Capacitors:C0603
- removed C21: 4.7uF, SparkFun-Capacitors:C0603
- removed C22: 10uF, SparkFun-Capacitors:C0603
- removed D2: 1A/23V/620mV, SparkFun-DiscreteSemi:SOD323
- removed LM2750: LM2750SD-5.0, LM2750SD-5.0:DFN300X300X80-11N
- removed LSM303: LSM303DLHC, LSM303DLHC:ST_LGA14_3X5
- removed MCP73831: MCP73831T-3ACI/OT, MCP73831T-3ACI_OT:SOT95P270X145-5N
- removed MOTOR+, MOTOR-, PIEZO+, PIEZO-: WIREPADSMD1,27-254, wirepad:SMD1,27-2,54
- removed PCA9555D: PCA9555, PCA9555:SO24-2
- removed R16: 330k, SparkFun-Resistors:R0603
- removed R46, R48: 1k, SparkFun-Resistors:R0603
- removed R47: 10k, SparkFun-Resistors:R0603
- removed SD-CARD: MF-MICROSD, MF_Connectors:MF-MICROSD
- removed TPS79533: TPS79533DCQR, TPS79533DCQR:SOT127P706X180-6N
- removed U$1: RYLED, myLib:RYLED
- removed U$2: L80GPS, myLib:L80GPS
- removed U$3: SKRHAAE010, HikeBuddy:ALPSSWITCH
- removed U$4: GPSNEO7M, HikeBuddy:GPSNEO7M
- removed U10, U12, U15, U8: (no value), MF_Discrete_Semiconductor:SOT-23-3
- removed U11: MF-DSC-SOT233-BSS84, MF_Discrete_Semiconductor:SOT-23-3
- added BATTERY1: (no value), SparkFun-Connectors:JST-2-SMD
- added C31: 33pF, MF_Passives:C0603
- added C32: 330pF, MF_Passives:C0603
- added C33: 10pF, MF_Passives:C0603
- added C34: 0.47uF, MF_Passives:C0603
- added C35: 0.1uF, MF_Passives:C0603
- added C36, C37: 4.7uF, SparkFun-Capacitors:C0603
- added C38, C39: 10uF, SparkFun-Capacitors:C0603
- added C40: 0.1uF, SparkFun-Capacitors:C0603
- added J5: SOLDER_PAD_2, SparkFun-Connectors:SOLDER_PAD_2
- added J6, J7: (no value), SparkFun-Connectors:1X01
- added J8: (no value), SparkFun-Connectors:1X06_LOCK
- added J9: 47352-1001, 47352-1001:MOLEX_47352-1001
- added L2: 3.3uH, LPS4018-472MRB:INDP_LPS4018-472MRB
- added L3, L5: 2.2uH, MF_Passives:L1210
- added L4, L6: 4.7uH, MF_Passives:L1210
- added S1, S2, S3, S4: B3U-3000P, B3U-3000P:SW_B3U-3000P
- added U1: LTC3586EUFE-1#PBF, LTC3586EUFE-3_TRPBF:QFN40P600X400X80-39N
- added U2: MAX17260SETD+, MAX17260SETD_coulomb:SON40P300X300X80-15N
- added U5: DRV2605LTDGSRQ1, DRV2605LTDGSRQ1:SOP50P490X110-10N
- added U7: LSM303CTR, LSM303CTR:LGA12R50P_200X200X100
- added UBLOX_GPS: CAM-M8C-0, CAM-M8C-0:LCC100P960X1400X210-31N
- added VREG_MODE: VREG MODE, jumper:SJ_2
- C10: value 10uF -> 0.1uF; device SparkFun-Capacitors:C0603 -> MF_Passives:C0603
- C11, C12, C30: value 1.0uF -> 22uF; device SparkFun-Capacitors:C0603 -> MF_Passives:C0603
- C13: value 10nF -> 10pF; device SparkFun-Capacitors:C0603 -> MF_Passives:C0603
- C16: value 4.7uF -> 10uF; device SparkFun-Capacitors:C0603 -> MF_Passives:C0603
- C17, C19: value 0.1uF -> 4.7uF
- C18: value 0.1uF -> 10pF; device SparkFun-Capacitors:C0603 -> MF_Passives:C0603
- C24: device SparkFun-Capacitors:C1206 -> MF_Passives:C0603
- C25: value 0.1uF -> 1uF; device SparkFun-Capacitors:C0603 -> MF_Passives:C0603
- C26: value 4.7uF -> 1uF; device SparkFun-Capacitors:C0603 -> MF_Passives:C0603
- C27: value 10nF -> 10uF; device SparkFun-Capacitors:C0603 -> MF_Passives:C0603
- C28: value 2.2uF -> 10uF; device SparkFun-Capacitors:C0603 -> MF_Passives:C0603
- C29: value 2.2uF -> 22uF; device SparkFun-Capacitors:C0603 -> MF_Passives:C0603
- C7: value 2.2uF -> 10uF
- C8: device SparkFun-Capacitors:C1206 -> SparkFun-Capacitors:C0603
- C9: value 2.2uF -> 10uF; device SparkFun-Capacitors:C0603 -> MF_Passives:C1206
- D1: value 1A/23V/620mV -> MF-LED-0603-RED; device SparkFun-DiscreteSemi:SOD323 -> MF_LEDs:LED0603
- FLASH, RESET: value MOMENTARY-SWITCH-SPST-SMD-5.2MM -> MF-SW-TACT-4.2MM; device SparkFun-Switches:TACTILE_SWITCH_SMD_5.2MM -> MF_Switches:TACT4.2MM
- FT231: value FT231XS-UTSSOP20 -> FT231XS
- J1: value 4P-SMD-2.0-90D -> MF-CON-MICROUSB-RIGHT; device OPL_Connector:HW4-SMD-2.0-90D -> MF_Connectors:MICROUSB-RIGHT
- J2: value 4P-2.0-90D -> GPS Port; device OPL_Connector:HW4-2.0-90D -> SparkFun-Connectors:1X06_LOCK
- J3: value MF-CON-MICROUSB-RIGHT -> (none); device MF_Connectors:MICROUSB-RIGHT -> SparkFun-Connectors:1X03_LOCK
- J4: value FH12-10S-0.5SH(1)(98) -> (none); device FH12-10S-0.5SH(1)(98):FH1210S05SH198 -> SparkFun-Connectors:1X03_LOCK
- R15: value 22 -> 100
- R17, R18, R19: value 10k -> 100
- R20: value 10k -> 100K; device SparkFun-Resistors:R0603 -> MF_Passives:R0603
- R21: value 10k -> 1K; device SparkFun-Resistors:R0603 -> MF_Passives:R0603
- R22: value 10k -> 220K; device SparkFun-Resistors:R0603 -> MF_Passives:R0603
- R23, R25, R26: value 10k -> 680K; device SparkFun-Resistors:R0603 -> MF_Passives:R0603
- R24: value 47k -> 220K; device SparkFun-Resistors:R0603 -> MF_Passives:R0603
- R27: value 200k -> 220K; device SparkFun-Resistors:R0603 -> MF_Passives:R0603
- R28: value 200k -> 121K; device SparkFun-Resistors:R0603 -> MF_Passives:R0603
- R29: value 22 -> 15K; device SparkFun-Resistors:R0603 -> MF_Passives:R0603
- R33, R34, R35, R36: value 1k -> 10k
- R37, R38: value 1k -> 2K
- R39: value 1k -> 750K
- R44: value 1k -> 560K
- R45: value 1k -> 100K
- R7: value 1k -> 2K; device SparkFun-Resistors:R0603 -> MF_Passives:R0603
- R8: value 1k -> 3K; device SparkFun-Resistors:R0603 -> MF_Passives:R0603
- R9: value 1k -> 560K; device SparkFun-Resistors:R0603 -> MF_Passives:R0603
- U$5: value FH12-10S-0.5SH -> 51441-1093
- U9: value MF-DSC-SOT233-BSS84 -> LTC6991CDCB#TRMPBF; device MF_Discrete_Semiconductor:SOT-23-3 -> LTC6991CS6TRMPBF:DFN
- moved D4 69.1 mm to (72.4, 4.08)
- moved C14 68.9 mm to (8.80, 14.1), flipped to the bottom, turned to 0 degrees
- moved J1 65.2 mm to (2.90, 31.6), turned to 270 degrees
- moved R13 65.1 mm to (8.70, 8.05), flipped to the bottom, turned to 180 degrees
- moved R12 65.0 mm to (8.70, 6.55), flipped to the bottom, turned to 180 degrees
- moved R43 65.0 mm to (8.72, 11.1), flipped to the bottom, turned to 180 degrees
- moved R14 64.8 mm to (8.70, 9.55), flipped to the bottom, turned to 180 degrees
- moved ANT 61.9 mm to (3.55, 0.60), flipped to the bottom, turned to 180 degrees
- moved R31 58.1 mm to (15.4, 14.2), flipped to the bottom, turned to 270 degrees
- moved C2 53.0 mm to (7.80, 4.30), flipped to the bottom, turned to 90 degrees
- moved C15 52.3 mm to (8.82, 12.6), flipped to the bottom, turned to 0 degrees
- moved J3 51.9 mm to (44.0, 38.5), turned to 0 degrees
- moved L1 50.9 mm to (10.3, 3.40), flipped to the bottom, turned to 0 degrees
- moved C16 50.3 mm to (10.2, 26.8), flipped to the bottom
- moved RESET 49.7 mm to (34.3, 30.2), turned to 180 degrees
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Connections:
- removed net 5V: C29.1, J4.6, J4.7, LM2750.1, LM2750.2, U$5.VDD, U$5.VDDA
- removed net AI1: C27.1, ESP32-PICO-D4.11, R27.1, R28.2
- removed net B1: PCA9555D.14, R33.1, U$3.P$1
- removed net B2: PCA9555D.15, R34.1, U$3.P$2
- removed net B3: PCA9555D.16, R35.1, U$3.P$3
- removed net B4: PCA9555D.13, R36.1, U$3.P$4
- removed net B5: PCA9555D.17, R39.1, U$3.P$6
- removed net DAC1: ESP32-PICO-D4.15, R30.2
- removed net DAC2: ESP32-PICO-D4.14, R32.2
- removed net GPIO_INT: ESP32-PICO-D4.24, PCA9555D.1, R48.1
- removed net GPS_POWER: D1.2, PCA9555D.7
- removed net IO12: R16.1, SD-CARD.PIN10, SD-CARD.PIN9
- removed net IO6: U$2.1PPS
- removed net IO7: ESP32-PICO-D4.10, MCP73831.1, U$1.R-, U$1.Y+
- removed net LCD_DISPLAY: J4.5, PCA9555D.9, U$5.DISP
- removed net LCD_POWER: LM2750.4, PCA9555D.10
- removed net N$24: C20.1, LSM303.P$13
- removed net N$25: C20.2, LSM303.P$12
- removed net N$36: R37.1, R46.1
- removed net RX_GPS: ESP32-PICO-D4.12, R20.2, U$2.TXD1, U$4.RX
- removed net SD_POWER: PCA9555D.8, R17.2
- removed net TX_GPS: ESP32-PICO-D4.13, R21.2, U$2.RXD1, U$4.TX
- removed net USB_DETECT: ESP32-PICO-D4.16, R25.1, R26.2
- removed net V_BATT: BATTERY.2, C10.1, C11.1, C28.1, LM2750.8, LM2750.9, MCP73831.3, R15.2, R27.2, R29.2, TPS79533.1, TPS79533.2, U$2.VBKP
- new net BAT_ALERT: U2.12
- new net EN_GPS: ESP32-PICO-D4.16, R31.2, U1.21
- new net EN_LCD: ESP32-PICO-D4.24, R36.2, U1.33
- new net EN_SDC: ESP32-PICO-D4.22, R30.2, U1.20
- new net GPS_RX: ESP32-PICO-D4.29, J2.5, R17.2
- new net GPS_SAFEBOOT: J2.3, R19.2
- new net GPS_TX: ESP32-PICO-D4.28, J2.4, R15.1
- new net HAP_EN: ESP32-PICO-D4.11, U5.5
- new net JUMPER: U1.9, VREG_MODE.2
- new net N$41: C36.1, U5.1
- new net N$42: R44.2, R45.1, U9.2
- new net N$43: C33.P$2, R29.P$2, U1.12
- new net N$44: C32.P$2, R29.P$1
- new net N$45: J9.1
- new net N$47: C34.P$2, U2.11
- new net N$50: J5.P$2, U5.9
- new net N$51: J5.P$1, U5.7
- new net SW1: ESP32-PICO-D4.5, R32.1, S1.2
- new net SW2: ESP32-PICO-D4.6, R33.1, S2.2
- new net SW3: ESP32-PICO-D4.7, R34.1, S3.2
- new net SW4: ESP32-PICO-D4.8, R35.1, S4.2
- new net V_BAT: BATTERY1.2, C35.P$2, C37.2, U1.32, U2.1, U2.10, U2.6, U2.7, U5.10, U5.6, UBLOX_GPS.8
- new net V_LCD: C11.P$2, C19.2, C29.P$2, J8.2, R44.1, R9.P$2, U$5.DISP, U$5.EXTMODE, U$5.VDD, U$5.VDDA, U1.6, U1.7, U9.1
- new net V_REG: C12.P$2, C25.P$2, C26.P$2, C27.P$2, C28.P$2, L2.1, L5.P$2, R21.P$2, U1.1, U1.14, U1.15, U1.18, U1.2, U1.22, U1.24, U1.27, U1.3, U1.34, VREG_MODE.3
- net 3V3_GPS: now also C13.P$1, C16.P$2, C17.1, J2.6, L4.P$1, R23.P$1, UBLOX_GPS.1, UBLOX_GPS.9; no longer C24.1, C25.1, C26.1, R19.1, R20.1, R21.1, U$2.VCC, U$4.VIN, U11.P$3
- net 3V3_SDC: now also C18.P$1, C24.P$1, J9.4, L6.P$2, R25.P$1; no longer C16.1, C17.1, C19.1, R16.2, R31.2, SD-CARD.PIN4, U9.P$3
- net ACCL1: now also ESP32-PICO-D4.13, U7.7; no longer LSM303.P$4, PCA9555D.18
- net ACCL2: now also ESP32-PICO-D4.12, U7.12; no longer LSM303.P$5, PCA9555D.19
- net D+: now also J1.3; no longer J3.3
- net D-: now also J1.2; no longer J3.2
- net ESP_EN: now also RESET.P$1, RESET.P$2; no longer RESET.3
- net ESP_FLASH: now also FLASH.P$1, FLASH.P$2, J4.3, J8.6; no longer FLASH.3
- net ESP_RX: now also J6.1
- net ESP_TX: now also J7.1
- net GND: now also BATTERY1.1, BATTERY1.NC1, BATTERY1.NC2, C10.P$1, C12.P$1, C16.P$1, C19.1, C24.P$2, C25.P$1, C26.P$1, C27.P$1, C28.P$1, C29.P$1, C30.P$2, C34.P$1, C35.P$1, C36.2, C37.1, C38.1, C39.2, C40.1, C8.1, C9.P$2, FLASH.P$3, FLASH.P$4, J1.5, J1.S1, J1.S2, J1.S3, J1.S4, J1.S5, J1.S6, J3.1, J4.1, J8.1, J9.6, J9.S1, J9.S2, J9.S3, J9.S4, R20.P$1, R22.P$2, R24.P$2, R27.P$1, R30.1, R31.1, R36.1, R39.2, R45.2, R7.P$1, R8.P$1, RESET.P$3, RESET.P$4, S1.1, S2.1, S3.1, S4.1, U1.39, U1.5, U2.15, U2.8, U2.9, U5.4, U5.8, U7.6, U7.8, U9.4, U9.5, U9.7, UBLOX_GPS.10, UBLOX_GPS.11, UBLOX_GPS.12, UBLOX_GPS.13, UBLOX_GPS.14, UBLOX_GPS.15, UBLOX_GPS.18, UBLOX_GPS.19, UBLOX_GPS.21, UBLOX_GPS.22, UBLOX_GPS.27, UBLOX_GPS.31, UBLOX_GPS.4, UBLOX_GPS.5, VREG_MODE.1; no longer BATTERY.1, C10.2, C11.2, C12.1, C13.1, C16.2, C18.2, C19.2, C21.1, C22.2, C24.2, C25.2, C26.2, C27.2, C28.2, C29.2, C8.2, C9.2, FLASH.1, J1.1, J3.5, J3.S1, J3.S2, J3.S3, J3.S4, J3.S5, J3.S6, J4.10, J4.11, J4.12, J4.8, J4.9, LM2750.11, LM2750.3, LM2750.5, LM2750.6, LSM303.P$10, LSM303.P$11, LSM303.P$7, MCP73831.2, PCA9555D.12, R26.1, R28.1, R44.1, R8.2, RESET.1, SD-CARD.G0, SD-CARD.G1, SD-CARD.PIN6, TPS79533.3, TPS79533.6, U$2.GND, U$2.GND2, U$3.P$5, U$4.GND, U$5.EXTMODE, U10.P$2, U12.P$2, U15.P$2, U8.P$2
- net GPS_RESET: now also J2.2, R18.2; no longer PCA9555D.11, R19.2, U$2.RESET
- net I2C_SCL: now also J3.2, R37.1, U2.14, U5.2, U7.1; no longer J1.4, J2.4, LSM303.P$2, PCA9555D.22, R46.2
- net I2C_SDA: now also J3.3, R38.1, U2.13, U5.3, U7.4; no longer J1.3, J2.3, LSM303.P$3, PCA9555D.23, R45.2
- net LCD_CLK: now also J8.5; no longer J4.1
- net LCD_CS: now also J8.3; no longer J4.3
- net LCD_MOSI: now also J8.4; no longer J4.2
- net LED1: now also ESP32-PICO-D4.18; no longer PCA9555D.6
- net LED2: now also ESP32-PICO-D4.15; no longer PCA9555D.4
- net LED3: now also ESP32-PICO-D4.14; no longer PCA9555D.5
- net MAGDRDY: now also ESP32-PICO-D4.10, U7.11; no longer LSM303.P$9, PCA9555D.20
- net N$10: now also R7.P$2, U1.29; no longer R8.1, U$1.Y-
- net N$11: now also C10.P$2, R8.P$2, U1.4; no longer R9.1, U$1.R+
- net N$12: now also C11.P$1, R20.P$2, R9.P$1, U1.10; no longer R22.1, U10.P$1
- net N$13: now also L3.P$2, U1.13; no longer MCP73831.5, R7.2
- net N$14: now also C31.P$1, C32.P$1, C33.P$1, R26.P$1, R27.P$2, U1.11; no longer C13.2, TPS79533.5
- net N$15: now also L2.2, U1.37; no longer R23.2, U10.P$3, U11.P$1
- net N$16: now also D1.CATHODE, U1.30; no longer D2.2, R24.1, U$2.TIMER
- net N$17: now also D1.ANODE, R21.P$1; no longer D1.1, D2.1, R22.2
- net N$18: now also L3.P$1, U1.19; no longer R30.1, U12.P$1
- net N$19: now also J9.8; no longer C21.2, LSM303.P$6
- net N$20: now also L4.P$2, U1.26; no longer R17.1, U8.P$1
- net N$21: now also C13.P$2, R22.P$1, R23.P$2, U1.28; no longer R18.2, U8.P$3, U9.P$1
- net N$22: now also L5.P$1, U1.8; no longer PIEZO+.1, R29.1
- net N$23: now also C40.2, U7.5; no longer R31.1, SD-CARD.PIN8
- net N$26: now also C18.P$2, R24.P$1, R25.P$2, U1.23; no longer PIEZO-.1, U12.P$3
- net N$27: now also L6.P$1, U1.25; no longer C30.1, LM2750.10
- net N$29: now also R15.2, UBLOX_GPS.25; no longer C30.2, LM2750.7
- net N$30: now also R17.1, UBLOX_GPS.26; no longer R32.1, U15.P$1
- net N$31: now also C31.P$2, R28.P$1; no longer R44.2, R7.1
- net N$34: now also UBLOX_GPS.16, UBLOX_GPS.17; no longer MOTOR+.1, R15.1
- net N$35: now also U$5.EXTCOMIN, U9.6; no longer R38.1, R45.1
- net N$37: now also R18.1, UBLOX_GPS.23; no longer MOTOR-.1, U15.P$3
- net N$38: now also R19.1, UBLOX_GPS.24; no longer R25.2, R47.1
- net N$40: now also R39.1, U9.3; no longer J4.4
- net SD_CLK: now also J9.5; no longer SD-CARD.PIN5
- net SD_CS: now also J9.2; no longer SD-CARD.PIN2
- net SD_MISO: now also J9.7; no longer SD-CARD.PIN7
- net SD_MOSI: now also J9.3; no longer SD-CARD.PIN3
- net VCC: now also C30.P$1, C38.2, C39.1, C8.2, J4.2, R26.P$2, R28.P$2, R32.2, U1.16, U1.17, U7.10, U7.2, U7.3, U7.9; no longer C12.2, C18.1, C22.1, C8.1, J1.2, J2.2, LSM303.P$1, LSM303.P$14, PCA9555D.2, PCA9555D.21, PCA9555D.24, PCA9555D.3, R18.1, R23.1, R24.2, R36.2, R39.2, R48.2, TPS79533.4, U11.P$2, U9.P$2
- net V_USB: now also C9.P$1, J1.1, U1.35, U1.36; no longer C9.1, J3.1, MCP73831.4, R47.2, R9.2
Routing:
- net V_BATT: track 125.4 -> 0.00 mm, vias 8 -> 0
- net V_BAT: track 0.00 -> 119.0 mm, vias 0 -> 5
- net 3V3_GPS: track 52.8 -> 147.8 mm, vias 2 -> 8
- net GND: track 413.8 -> 505.9 mm, vias 27 -> 95
- net SW2: track 0.00 -> 89.5 mm, vias 0 -> 2
- net USB_DETECT: track 81.8 -> 0.00 mm, vias 1 -> 0
- net SW4: track 0.00 -> 72.1 mm, vias 0 -> 3
- net GPS_TX: track 0.00 -> 70.9 mm, vias 0 -> 3
- net GPS_RX: track 0.00 -> 70.3 mm, vias 0 -> 3
- net IO7: track 69.3 -> 0.00 mm, vias 4 -> 0
- net SW1: track 0.00 -> 68.6 mm, vias 0 -> 4
- net RX_GPS: track 63.6 -> 0.00 mm, vias 1 -> 0
- net VCC: track 299.8 -> 236.3 mm, vias 16 -> 18
- net TX_GPS: track 61.0 -> 0.00 mm, vias 1 -> 0
- net SW3: track 0.00 -> 59.2 mm, vias 0 -> 3
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- added copper zone on layer 1, net GND
- added copper zone on layer 16, net GND
- added copper zone on layer 1, net VCC
- added copper zone on layer 16, net V_BAT
- added copper zone on layer 1, net V_REG
Other:
- board size 80 x 40 mm -> 75 x 40 mm
- board text added: "2020 Saurabh Gandhi"
- board text added: "ESP_RX"
- board text added: "ESP_TX"
- board text added: "GPIO/ Flash"
- board text added: "GPIO0/ FLASH"
- board text added: "GPIO13"
- board text added: "GPIO14"
- board text added: "GPIO15"
- board text added: "GPS / UART Extension"
- board text added: "I2C Extension"
- board text added: "LCD / GPIO Extension"
- board text added: "RESET"
- board text added: "SAFEBOOT"
- board text added: "VCC (LCD)"
- board text added: "V_GPS (3.3V)"
- board text removed: "2019 Saurabh Gandhi"
- board text removed: "3V3"
- board text removed: "CHG STAT"
- board text removed: "FT231"
- board text removed: "GROVE I2C connector"
- board text removed: "LM2750"
- board text removed: "LSM303"
- board text removed: "MCP73831"
- board text removed: "TPS79533"
- board text removed: "UART connector (on-board GPS module)"
- board text removed: "USB"

Commit message: updates
Parts:
- U7: device LSM303CTR:LGA12R50P_200X200X100 -> LSM303CTR:LGA-12
Routing:
- net VCC: track 236.3 -> 235.5 mm
