File: Hardware/hikebuddy_dhauladhar/base.sch (EAGLE design)
At the start: 116 parts, among them J1 4P-SMD-2.0-90D, J2 4P-2.0-90D, J3 MF-CON-MICROUSB-RIGHT, J4 FH12-10S-0.5SH(1)(98), U11 MF-DSC-SOT233-BSS84, U3 MF-DSC-SOT233-MMBT3904, U4 MF-DSC-SOT233-MMBT3904, U9 MF-DSC-SOT233-BSS84

Commit message: last commit before starting V2
Changed lines of the file:
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@@
 <?xml version="1.0" encoding="utf-8"?>
 <!DOCTYPE eagle SYSTEM "eagle.dtd">
-<eagle version="9.3.1">
+<eagle version="9.5.1">
 <drawing>
 <settings>
-<setting alwaysvectorfont="yes"/>
+<setting alwaysvectorfont="no"/>
 <setting verticaltext="up"/>
 </settings>
@@
 <part name="GND25" library="supply1" library_urn="urn:adsk.eagle:library:371" deviceset="GND" device=""/>
 <part name="R30" library="SparkFun-Resistors" deviceset="10KOHM" device="-0603-1/10W-1%" package3d_urn="urn:adsk.eagle:package:23555/3" value="10k"/>
-<part name="PIEZO+" library="wirepad" library_urn="urn:adsk.eagle:library:412" deviceset="WIREPAD" device="SMD1,27-254" package3d_urn="urn:adsk.eagle:package:30839/1" value=""/>
-<part name="PIEZO-" library="wirepad" library_urn="urn:adsk.eagle:library:412" deviceset="WIREPAD" device="SMD1,27-254" package3d_urn="urn:adsk.eagle:package:30839/1" value=""/>
+<part name="PIEZO+" library="wirepad" library_urn="urn:adsk.eagle:library:412" deviceset="WIREPAD" device="SMD1,27-254" package3d_urn="urn:adsk.eagle:package:30839/1" value="WIREPADSMD1,27-254"/>
+<part name="PIEZO-" library="wirepad" library_urn="urn:adsk.eagle:library:412" deviceset="WIREPAD" device="SMD1,27-254" package3d_urn="urn:adsk.eagle:package:30839/1" value="WIREPADSMD1,27-254"/>
 <part name="SUPPLY9" library="SparkFun-PowerSymbols" library_urn="urn:adsk.eagle:library:530" deviceset="V_BATT" device=""/>
 <part name="LM2750" library="LM2750SD-5.0" deviceset="LM2750SD-5.0" device="" package3d_urn="urn:adsk.eagle:package:9987730/3"/>
@@
 <part name="GND32" library="supply1" library_urn="urn:adsk.eagle:library:371" deviceset="GND" device=""/>
 <part name="R32" library="SparkFun-Resistors" deviceset="10KOHM" device="-0603-1/10W-1%" package3d_urn="urn:adsk.eagle:package:23555/3" value="10k"/>
-<part name="MOTOR+" library="wirepad" library_urn="urn:adsk.eagle:library:412" deviceset="WIREPAD" device="SMD1,27-254" package3d_urn="urn:adsk.eagle:package:30839/1" value=""/>
-<part name="MOTOR-" library="wirepad" library_urn="urn:adsk.eagle:library:412" deviceset="WIREPAD" device="SMD1,27-254" package3d_urn="urn:adsk.eagle:package:30839/1" value=""/>
+<part name="MOTOR+" library="wirepad" library_urn="urn:adsk.eagle:library:412" deviceset="WIREPAD" device="SMD1,27-254" package3d_urn="urn:adsk.eagle:package:30839/1" value="WIREPADSMD1,27-254"/>
+<part name="MOTOR-" library="wirepad" library_urn="urn:adsk.eagle:library:412" deviceset="WIREPAD" device="SMD1,27-254" package3d_urn="urn:adsk.eagle:package:30839/1" value="WIREPADSMD1,27-254"/>
 <part name="SUPPLY12" library="SparkFun-PowerSymbols" library_urn="urn:adsk.eagle:library:530" deviceset="V_BATT" device=""/>
 <part name="R33" library="SparkFun-Resistors" deviceset="1KOHM" device="-0603-1/10W-1%" package3d_urn="urn:adsk.eagle:package:23555/3" value="1k"/>

Commit message: digikey_cs_v0
Parts:
- removed BATTERY: (no value), SparkFun-Connectors:JST_2MM_MALE
- removed C20: 0.22uF, SparkFun-Capacitors:0.22UF-0603-25V-10%
- removed C21: 4.7uF, SparkFun-Capacitors:4.7UF-0603-6.3V-(10%)
- removed C22: 10uF, SparkFun-Capacitors:10UF-0603-6.3V-20%
- removed D2: 1A/23V/620mV, SparkFun-DiscreteSemi:DIODE-SCHOTTKY-BAT20J
- removed LM2750: LM2750SD-5.0, LM2750SD-5.0:LM2750SD-5.0
- removed LSM303: LSM303DLHC, LSM303DLHC:LSM303DLHC
- removed MCP73831: MCP73831T-3ACI/OT, MCP73831T-3ACI_OT:MCP73831T-3ACI/OT
- removed MOTOR+, MOTOR-, PIEZO+, PIEZO-: WIREPADSMD1,27-254, wirepad:WIREPADSMD1,27-254
- removed PCA9555D: PCA9555, PCA9555:PCA9555
- removed R16: 330k, SparkFun-Resistors:330KOHM-0603-1/10W-1%
- removed R46, R48: 1k, SparkFun-Resistors:1KOHM-0603-1/10W-1%
- removed R47: 10k, SparkFun-Resistors:10KOHM-0603-1/10W-1%
- removed SD-CARD: MF-MICROSD, MF_Connectors:SD_CARD_SLOT_MICRO_RIGHT
- removed TPS79533: TPS79533DCQR, TPS79533DCQR:TPS79533DCQR
- removed U$1: RYLED, myLib:RYLED
- removed U$2: L80GPS, myLib:L80GPS
- removed U$3: SKRHAAE010, HikeBuddy:ALPSSWITCH
- removed U$4: GPSNEO7M, HikeBuddy:GPSNEO7M
- removed U10, U12, U15, U8: (no value), MF_Discrete_Semiconductor:NPN_BJT_SOT-23-3
- removed U11: MF-DSC-SOT233-BSS84, MF_Discrete_Semiconductor:P-CHANNEL_FET_BSS84_SOT-23-3
- added BATTERY1: (no value), SparkFun-Connectors:JST_2MM_MALE
- added C31: 33pF, MF_Passives:CAPACITOR_NP_0603
- added C32: 330pF, MF_Passives:CAPACITOR_NP_0603
- added C33: 10pF, MF_Passives:CAPACITOR_NP_0603
- added C34: 0.47uF, MF_Passives:CAPACITOR_NP_0603
- added C35: 0.1uF, MF_Passives:CAPACITOR_NP_0603
- added C36, C37: 4.7uF, SparkFun-Capacitors:4.7UF-0603-6.3V-(10%)
- added C38: 10uF, SparkFun-Capacitors:4.7PF-0603-50V-5%
- added C39: 10uF, SparkFun-Capacitors:10UF-0603-6.3V-20%
- added C40: 0.1uF, SparkFun-Capacitors:4.7UF-0603-6.3V-(10%)
- added J5: SOLDER_PAD_2, SparkFun-Connectors:SOLDER_PAD_2
- added J6, J7: (no value), SparkFun-Connectors:CONN_01
- added J8: (no value), SparkFun-Connectors:CONN_06LOCK
- added J9: 47352-1001, 47352-1001:47352-1001
- added L2: 3.3uH, LPS4018-472MRB:LPS4018-472MRB
- added L3, L5: 2.2uH, MF_Passives:INDUCTOR_1210
- added L4, L6: 4.7uH, MF_Passives:INDUCTOR_1210
- added S1, S2, S3, S4: B3U-3000P, B3U-3000P:B3U-3000P
- added U1: LTC3586EUFE-1#PBF, LTC3586EUFE-3_TRPBF:LTC3586EUFE-3#TRPBF
- added U2: MAX17260SETD+, MAX17260SETD_coulomb:MAX17260SETD+
- added U5: DRV2605LTDGSRQ1, DRV2605LTDGSRQ1:DRV2605LTDGSRQ1
- added U7: LSM303CTR, LSM303CTR:LSM303CTR
- added UBLOX_GPS: CAM-M8C-0, CAM-M8C-0:CAM-M8C-0
- added VREG_MODE: VREG MODE, jumper:SJ2W
- C10: value 10uF -> 0.1uF; device SparkFun-Capacitors:10UF-0603-6.3V-20% -> MF_Passives:CAPACITOR_NP_0603
- C11, C12, C30: value 1.0uF -> 22uF; device SparkFun-Capacitors:1.0UF-0603-16V-10% -> MF_Passives:CAPACITOR_NP_0603
- C13: value 10nF -> 10pF; device SparkFun-Capacitors:10NF-0603-50V-10% -> MF_Passives:CAPACITOR_NP_0603
- C16: value 4.7uF -> 10uF; device SparkFun-Capacitors:4.7UF-0603-6.3V-(10%) -> MF_Passives:CAPACITOR_NP_0603
- C17: value 0.1uF -> 4.7uF
- C18: value 0.1uF -> 10pF; device SparkFun-Capacitors:0.1UF-0603-25V-5% -> MF_Passives:CAPACITOR_NP_0603
- C19: value 0.1uF -> 4.7uF; device SparkFun-Capacitors:0.1UF-0603-25V-5% -> SparkFun-Capacitors:4.7UF-0603-6.3V-(10%)
- C24: device SparkFun-Capacitors:10UF-1206-6.3V-20% -> MF_Passives:CAPACITOR_NP_0603
- C25: value 0.1uF -> 1uF; device SparkFun-Capacitors:0.1UF-0603-25V-5% -> MF_Passives:CAPACITOR_NP_0603
- C26: value 4.7uF -> 1uF; device SparkFun-Capacitors:4.7UF-0603-6.3V-(10%) -> MF_Passives:CAPACITOR_NP_0603
- C27: value 10nF -> 10uF; device SparkFun-Capacitors:10NF-0603-50V-10% -> MF_Passives:CAPACITOR_NP_0603
- C28: value 2.2uF -> 10uF; device SparkFun-Capacitors:2.2UF-0603-10V-20% -> MF_Passives:CAPACITOR_NP_0603
- C29: value 2.2uF -> 22uF; device SparkFun-Capacitors:2.2UF-0603-10V-20% -> MF_Passives:CAPACITOR_NP_0603
- C7: value 2.2uF -> 10uF
- C8: device SparkFun-Capacitors:10UF-1206-6.3V-20% -> SparkFun-Capacitors:4.7PF-0603-50V-5%
- C9: value 2.2uF -> 10uF; device SparkFun-Capacitors:2.2UF-0603-10V-20% -> MF_Passives:CAPACITOR_NP_1206
- D1: value 1A/23V/620mV -> MF-LED-0603-RED; device SparkFun-DiscreteSemi:DIODE-SCHOTTKY-BAT20J -> MF_LEDs:LED_SINGLE-0603-RED
- FLASH, RESET: value MOMENTARY-SWITCH-SPST-SMD-5.2MM -> MF-SW-TACT-4.2MM; device SparkFun-Switches:MOMENTARY-SWITCH-SPST-SMD-5.2MM -> MF_Switches:TACT_4.2MM
- FT231: value FT231XS-UTSSOP20 -> FT231XS
- J1: value 4P-SMD-2.0-90D -> MF-CON-MICROUSB-RIGHT; device OPL_Connector:GROVE-CONNECTOR-SMD-90D(4+2P-2.0) -> MF_Connectors:USB_MICRO_RIGHT
- J2: value 4P-2.0-90D -> GPS Port; device OPL_Connector:GROVE-CONNECTOR-DIP-90D(4P-2.0) -> SparkFun-Connectors:CONN_06LOCK
- J3: value MF-CON-MICROUSB-RIGHT -> (none); device MF_Connectors:USB_MICRO_RIGHT -> SparkFun-Connectors:CONN_03LOCK
- J4: value FH12-10S-0.5SH(1)(98) -> (none); device FH12-10S-0.5SH(1)(98):FH12-10S-0.5SH(1)(98) -> SparkFun-Connectors:CONN_03LOCK
- L1: MPN (none) -> 744761016C
- R15: value 22 -> 100; device SparkFun-Resistors:22OHM-0603-1/10W-1% -> SparkFun-Resistors:1KOHM-0603-1/10W-1%
- R17: value 10k -> 100; device SparkFun-Resistors:10KOHM-0603-1/10W-1% -> SparkFun-Resistors:1KOHM-0603-1/10W-1%
- R18, R19: value 10k -> 100; device SparkFun-Resistors:10KOHM-0603-1/10W-1% -> SparkFun-Resistors:1KOHM-0603-1/10W-1%; DNP (none) -> 1
- R20: value 10k -> 100K; device SparkFun-Resistors:10KOHM-0603-1/10W-1% -> MF_Passives:RESISTOR_0603
- R21: value 10k -> 1K; device SparkFun-Resistors:10KOHM-0603-1/10W-1% -> MF_Passives:RESISTOR_0603
- R22: value 10k -> 220K; device SparkFun-Resistors:10KOHM-0603-1/10W-1% -> MF_Passives:RESISTOR_0603
- R23, R25, R26: value 10k -> 680K; device SparkFun-Resistors:10KOHM-0603-1/10W-1% -> MF_Passives:RESISTOR_0603
- R24: value 47k -> 220K; device SparkFun-Resistors:47KOHM-0603-1/10W-1% -> MF_Passives:RESISTOR_0603
- R27: value 200k -> 220K; device SparkFun-Resistors:200KOHM-0603-1/10W-1% -> MF_Passives:RESISTOR_0603
- R28: value 200k -> 121K; device SparkFun-Resistors:200KOHM-0603-1/10W-1% -> MF_Passives:RESISTOR_0603
- R29: value 22 -> 15K; device SparkFun-Resistors:22OHM-0603-1/10W-1% -> MF_Passives:RESISTOR_0603
- R33, R34, R35, R36: value 1k -> 10k; device SparkFun-Resistors:1KOHM-0603-1/10W-1% -> SparkFun-Resistors:10KOHM-0603-1/10W-1%
- R37, R38: value 1k -> 2K
- R39: value 1k -> 750K
- R44: value 1k -> 560K
- R45: value 1k -> 100K
- R7: value 1k -> 2K; device SparkFun-Resistors:1KOHM-0603-1/10W-1% -> MF_Passives:RESISTOR_0603
- R8: value 1k -> 3K; device SparkFun-Resistors:1KOHM-0603-1/10W-1% -> MF_Passives:RESISTOR_0603
- R9: value 1k -> 560K; device SparkFun-Resistors:1KOHM-0603-1/10W-1% -> MF_Passives:RESISTOR_0603
- U$5: value FH12-10S-0.5SH -> 51441-1093; MPN (none) -> 51441-1093
- U9: value MF-DSC-SOT233-BSS84 -> LTC6991CDCB#TRMPBF; device MF_Discrete_Semiconductor:P-CHANNEL_FET_BSS84_SOT-23-3 -> LTC6991CS6TRMPBF:LTC6991CS6TRMPBFDFN
Connections:
- removed net 5V: C29.1, J4.6, J4.7, LM2750.VOUT, LM2750.VOUT_2, U$5.VDD, U$5.VDDA
- removed net AI1: C27.1, ESP32-PICO-D4.IO35, R27.1, R28.2
- removed net B1: PCA9555D.I/O1.1, R33.1, U$3.A
- removed net B2: PCA9555D.I/O1.2, R34.1, U$3.CENTER
- removed net B3: PCA9555D.I/O1.3, R35.1, U$3.C
- removed net B4: PCA9555D.I/O1.0, R36.1, U$3.B
- removed net B5: PCA9555D.I/O1.4, R39.1, U$3.D
- removed net DAC1: ESP32-PICO-D4.IO26, R30.2
- removed net DAC2: ESP32-PICO-D4.IO25, R32.2
- removed net GPIO_INT: ESP32-PICO-D4.IO4, PCA9555D.!INT, R48.1
- removed net GPS_POWER: D1.A, PCA9555D.I/O0.3
- removed net IO12: R16.1, SD-CARD.CRD_DTCT
- removed net IO6: U$2.1PPS
- removed net IO7: ESP32-PICO-D4.IO34, MCP73831.STAT, U$1.P$1, U$1.P$3
- removed net LCD_DISPLAY: J4.5, PCA9555D.I/O0.5, U$5.DISP
- removed net LCD_POWER: LM2750.SD, PCA9555D.I/O0.6
- removed net N$24: C20.1, LSM303.SETC
- removed net N$25: C20.2, LSM303.SETP
- removed net N$36: R37.1, R46.1
- removed net RX_GPS: ESP32-PICO-D4.IO32, R20.2, U$2.TX, U$4.RX
- removed net SD_POWER: PCA9555D.I/O0.4, R17.2
- removed net TX_GPS: ESP32-PICO-D4.IO33, R21.2, U$2.RX, U$4.TX
- removed net USB_DETECT: ESP32-PICO-D4.IO27, R25.1, R26.2
- removed net V_BATT: BATTERY.+, C10.1, C11.1, C28.1, LM2750.VIN, LM2750.VIN_2, MCP73831.VBAT, R15.2, R27.2, R29.2, TPS79533.EN, TPS79533.IN, U$2.VBKP
- new net BAT_ALERT: U2.ALRT
- new net EN_GPS: ESP32-PICO-D4.IO27, R31.2, U1.EN1
- new net EN_LCD: ESP32-PICO-D4.IO4, R36.2, U1.EN4
- new net EN_SDC: ESP32-PICO-D4.IO2, R30.2, U1.EN2
- new net GPS_RX: ESP32-PICO-D4.SD3, J2.5, R17.2
- new net GPS_SAFEBOOT: J2.3, R19.2
- new net GPS_TX: ESP32-PICO-D4.SD2, J2.4, R15.1
- new net HAP_EN: ESP32-PICO-D4.IO35, U5.EN
- new net JUMPER: U1.MODE, VREG_MODE.2
- new net N$41: C36.1, U5.REG
- new net N$42: R44.2, R45.1, U9.DIV
- new net N$43: C33.P$2, R29.P$2, U1.VC3
- new net N$44: C32.P$2, R29.P$1
- new net N$45: J9.DATA2
- new net N$47: C34.P$2, U2.REG
- new net N$50: J5.2, U5.OUT-
- new net N$51: J5.1, U5.OUT+
- new net SW1: ESP32-PICO-D4.SENSOR_VP, R32.1, S1.2
- new net SW2: ESP32-PICO-D4.SENSOR_CAPP, R33.1, S2.2
- new net SW3: ESP32-PICO-D4.SENSOR_CAPN, R34.1, S3.2
- new net SW4: ESP32-PICO-D4.SENSOR_VN, R35.1, S4.2
- new net V_BAT: BATTERY1.+, C35.P$2, C37.2, U1.BAT, U2.BATT, U2.CSN, U2.CSPH, U2.TH, U5.VDD, U5.VDD/NC, UBLOX_GPS.V_BCKP
- new net V_LCD: C11.P$2, C19.2, C29.P$2, J8.2, R44.1, R9.P$2, U$5.DISP, U$5.EXTMODE, U$5.VDD, U$5.VDDA, U1.VOUT4, U9.V+
- new net V_REG: C12.P$2, C25.P$2, C26.P$2, C27.P$2, C28.P$2, L2.1, L5.P$2, R21.P$2, U1.EN3, U1.ILIM0, U1.ILIM1, U1.LDO3V3, U1.VIN1, U1.VIN2, U1.VIN3, U1.VIN4, U1.VOUT, VREG_MODE.3
- net 3V3_GPS: now also C13.P$1, C16.P$2, C17.1, J2.6, L4.P$1, R23.P$1, UBLOX_GPS.VCC, UBLOX_GPS.VCC_IO; no longer C24.1, C25.1, C26.1, R19.1, R20.1, R21.1, U$2.VCC, U$4.VIN, U11.DRAIN
- net 3V3_SDC: now also C18.P$1, C24.P$1, J9.VDD, L6.P$2, R25.P$1; no longer C16.1, C17.1, C19.1, R16.2, R31.2, SD-CARD.3.3V, U9.DRAIN
- net ACCL1: now also ESP32-PICO-D4.IO33, U7.INT_MAG; no longer LSM303.INT2, PCA9555D.I/O1.5
- net ACCL2: now also ESP32-PICO-D4.IO32, U7.INT_XL; no longer LSM303.INT1, PCA9555D.I/O1.6
- net D+: now also J1.D+; no longer J3.D+
- net D-: now also J1.D-; no longer J3.D-
- net ESP_EN: now also RESET.P$1, RESET.P$2; no longer RESET.2
- net ESP_FLASH: now also FLASH.P$1, FLASH.P$2, J4.3, J8.6; no longer FLASH.2
- net ESP_RX: now also J6.1
- net ESP_TX: now also J7.1
- net GND: now also BATTERY1.-, BATTERY1.PAD1, BATTERY1.PAD2, C10.P$1, C12.P$1, C16.P$1, C19.1, C24.P$2, C25.P$1, C26.P$1, C27.P$1, C28.P$1, C29.P$1, C30.P$2, C34.P$1, C35.P$1, C36.2, C37.1, C38.1, C39.2, C40.1, C8.1, C9.P$2, FLASH.P$3, FLASH.P$4, J1.GND, J1.SLD, J3.1, J4.1, J8.1, J9.SHIELD, J9.VSS, R20.P$1, R22.P$2, R24.P$2, R27.P$1, R30.1, R31.1, R36.1, R39.2, R45.2, R7.P$1, R8.P$1, RESET.P$3, RESET.P$4, S1.1, S2.1, S3.1, S4.1, U1.GND, U1.NTC, U2.CSPL, U2.EP, U2.GND, U5.GND, U5.IN/TRIG, U7.GND, U9.GND, U9.RST, UBLOX_GPS.GND, UBLOX_GPS.GND-1, UBLOX_GPS.GND-10, UBLOX_GPS.GND-11, UBLOX_GPS.GND-12, UBLOX_GPS.GND-13, UBLOX_GPS.GND-2, UBLOX_GPS.GND-3, UBLOX_GPS.GND-4, UBLOX_GPS.GND-5, UBLOX_GPS.GND-6, UBLOX_GPS.GND-7, UBLOX_GPS.GND-8, UBLOX_GPS.GND-9, VREG_MODE.1; no longer BATTERY.-, C10.2, C11.2, C12.1, C13.1, C16.2, C18.2, C19.2, C21.1, C22.2, C24.2, C25.2, C26.2, C27.2, C28.2, C29.2, C8.2, C9.2, FLASH.1, J1.1, J3.GND, J3.SLD, J4.10, J4.11, J4.12, J4.8, J4.9, LM2750.FB, LM2750.GND, LM2750.GND_2, LM2750.GND_3, LSM303.GND, LSM303.RES@2, LSM303.RES@3, MCP73831.VSS, PCA9555D.VSS, R26.1, R28.1, R44.1, R8.2, RESET.1, SD-CARD.GND, TPS79533.GND_1, TPS79533.GND_2, U$2.GND, U$3.GND, U$4.GND, U$5.EXTMODE, U10.EMITTER, U12.EMITTER, U15.EMITTER, U8.EMITTER
- net GPS_RESET: now also J2.2, R18.2; no longer PCA9555D.I/O0.7, R19.2, U$2.RESET
- net I2C_SCL: now also J3.2, R37.1, U2.SCL, U5.SCL, U7.SCL/SPC; no longer J1.4, J2.4, LSM303.SCL, PCA9555D.SCL, R46.2
- net I2C_SDA: now also J3.3, R38.1, U2.SDA, U5.SDA, U7.SDA/SDI/SDO; no longer J1.3, J2.3, LSM303.SDA, PCA9555D.SDA, R45.2
- net LCD_CLK: now also J8.5; no longer J4.1
- net LCD_CS: now also J8.3; no longer J4.3
- net LCD_MOSI: now also J8.4; no longer J4.2
- net LED1: now also ESP32-PICO-D4.IO12; no longer PCA9555D.I/O0.2
- net LED2: now also ESP32-PICO-D4.IO26; no longer PCA9555D.I/O0.0
- net LED3: now also ESP32-PICO-D4.IO25; no longer PCA9555D.I/O0.1
- net MAGDRDY: now also ESP32-PICO-D4.IO34, U7.DRDY_MAG; no longer LSM303.DRDY, PCA9555D.I/O1.7
- net N$10: now also R7.P$2, U1.PROG; no longer R8.1, U$1.P$2
- net N$11: now also C10.P$2, R8.P$2, U1.CLPROG; no longer R9.1, U$1.P$4
- net N$12: now also C11.P$1, R20.P$2, R9.P$1, U1.FB4; no longer R22.1, U10.BASE
- net N$13: now also L3.P$2, U1.SWAB3; no longer MCP73831.PROG, R7.2
- net N$14: now also C31.P$1, C32.P$1, C33.P$1, R26.P$1, R27.P$2, U1.FB3; no longer C13.2, TPS79533.FB
- net N$15: now also L2.2, U1.SW; no longer R23.2, U10.COLLECTOR, U11.GATE
- net N$16: now also D1.CATHODE, U1.CHRG; no longer D2.A, R24.1, U$2.TIMER
- net N$17: now also D1.ANODE, R21.P$1; no longer D1.C, D2.C, R22.2
- net N$18: now also L3.P$1, U1.SWCD3; no longer R30.1, U12.BASE
- net N$19: now also J9.DATA1; no longer C21.2, LSM303.C1
- net N$20: now also L4.P$2, U1.SW1; no longer R17.1, U8.BASE
- net N$21: now also C13.P$2, R22.P$1, R23.P$2, U1.FB1; no longer R18.2, U8.COLLECTOR, U9.GATE
- net N$22: now also L5.P$1, U1.SW4; no longer PIEZO+.P, R29.1
- net N$23: now also C40.2, U7.C1; no longer R31.1, SD-CARD.IRQ
- net N$26: now also C18.P$2, R24.P$1, R25.P$2, U1.FB2; no longer PIEZO-.P, U12.COLLECTOR
- net N$27: now also L6.P$1, U1.SW2; no longer C30.1, LM2750.C+
- net N$29: now also R15.2, UBLOX_GPS.TXD/SPI_MISO; no longer C30.2, LM2750.C-
- net N$30: now also R17.1, UBLOX_GPS.RXD/SPI_MOSI; no longer R32.1, U15.BASE
- net N$31: now also C31.P$2, R28.P$1; no longer R44.2, R7.1
- net N$34: now also UBLOX_GPS.RF_IN, UBLOX_GPS.RF_OUT; no longer MOTOR+.P, R15.1
- net N$35: now also U$5.EXTCOMIN, U9.OUT; no longer R38.1, R45.1
- net N$37: now also R18.1, UBLOX_GPS.RESET_N; no longer MOTOR-.P, U15.COLLECTOR
- net N$38: now also R19.1, UBLOX_GPS.SAFEBOOT_N; no longer R25.2, R47.1
- net N$40: now also R39.1, U9.SET; no longer J4.4
- net SD_CLK: now also J9.CLK; no longer SD-CARD.SCLK
- net SD_CS: now also J9.CD/DATA3; no longer SD-CARD.CS
- net SD_MISO: now also J9.DATA0; no longer SD-CARD.D0
- net SD_MOSI: now also J9.CMD; no longer SD-CARD.DI
- net VCC: now also C30.P$1, C38.2, C39.1, C8.2, J4.2, R26.P$2, R28.P$2, R32.2, U1.VOUT3, U7.CS_MAG, U7.CS_XL, U7.VDD, U7.VDD_IO; no longer C12.2, C18.1, C22.1, C8.1, J1.2, J2.2, LSM303.VDD, LSM303.VDDIO, PCA9555D.A0, PCA9555D.A1, PCA9555D.A2, PCA9555D.VDD, R18.1, R23.1, R24.2, R36.2, R39.2, R48.2, TPS79533.OUT, U11.SOURCE, U9.SOURCE
- net V_USB: now also C9.P$1, J1.5V, U1.VBUS; no longer C9.1, J3.5V, MCP73831.VIN, R47.2, R9.2
Other:
- note removed: "GPIO2 and GPIO12 must be low at power-up."
